File: doc/Schaltplan/RFID_Controller.brd (EAGLE design)
At the start: 77 x 67 mm, 42 parts, among them IC2 MCP23017SP, K1 FTR-K1C, T1 BC547, T2 BC547

Commit message: -mod: fixed a bug in the schematic/layout
Connections:
- new net N$9: IC2.2, R15.2
- net SW: no longer IC2.2, R15.2
Routing:
- net SW: track 25.7 -> 14.4 mm
- net N$9: track 0.00 -> 8.65 mm
Changed lines of the file:
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@@
 <signal name="SW">
 <contactref element="R10" pad="2"/>
-<contactref element="IC2" pad="2"/>
 <contactref element="T1" pad="2"/>
-<contactref element="R15" pad="2"/>
 <contactref element="R5" pad="1"/>
-<wire x1="48.514" y1="38.1" x2="50.546" y2="38.1" width="1.016" layer="16"/>
-<wire x1="50.546" y1="38.1" x2="52.07" y2="39.624" width="1.016" layer="16"/>
-<wire x1="52.07" y1="39.624" x2="52.07" y2="43.942" width="1.016" layer="16"/>
-<wire x1="52.07" y1="43.942" x2="52.07" y2="46.736" width="1.016" layer="16"/>
 <wire x1="52.07" y1="46.736" x2="50.8" y2="46.736" width="1.016" layer="16"/>
 <wire x1="50.8" y1="46.736" x2="48.006" y2="49.53" width="1.016" layer="16"/>
@@
 <wire x1="44.45" y1="46.736" x2="44.45" y2="43.942" width="1.016" layer="16"/>
 </signal>
+<signal name="N$9">
+<contactref element="R15" pad="2"/>
+<contactref element="IC2" pad="2"/>
+<wire x1="48.514" y1="38.1" x2="50.8" y2="38.1" width="1.016" layer="16"/>
+<wire x1="50.8" y1="38.1" x2="52.07" y2="39.37" width="1.016" layer="16"/>
+<wire x1="52.07" y1="39.37" x2="52.07" y2="43.942" width="1.016" layer="16"/>
+</signal>
 </signals>
