File: doc/Schaltplan/RFID_Controller.sch (EAGLE design)
At the start: 42 parts, among them IC2 MCP23017SP, K1 FTR-K1C, T1 BC547, T2 BC547

Commit message: -mod: fixed a bug in the schematic/layout
Connections:
- new net N$9: IC2.GPB1, R15.2
- net SW: no longer IC2.GPB1, R15.2
Changed lines of the file:
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@@
-</segment>
-<segment>
-<pinref part="IC2" gate="G$1" pin="GPB1"/>
-<wire x1="160.02" y1="71.12" x2="162.56" y2="71.12" width="0.1524" layer="91"/>
-<pinref part="R15" gate="G$1" pin="2"/>
 </segment>
 <segment>
@@
 </segment>
 </net>
+<net name="N$9" class="0">
+<segment>
+<pinref part="R15" gate="G$1" pin="2"/>
+<pinref part="IC2" gate="G$1" pin="GPB1"/>
+<wire x1="162.56" y1="71.12" x2="160.02" y2="71.12" width="0.1524" layer="91"/>
+</segment>
+</net>
